File: LockSequencer.brd (EAGLE design)
At the start: 80.3 x 77.5 mm, 76 parts, among them IC1 4017D, IC2 NE555, K1 G2RATE-OJ, K2 G2RATE-OJ

Commit message: Final tweaks to layout
Parts:
- added H1, H2: MOUNT-HOLE3.0, holes:3,0
- moved C1 5.12 mm to (34.3, 59.7), turned to 45 degrees
- moved T3 2.01 mm to (46.4, 15.2)
- moved D11 1.27 mm to (58.4, 12.7)
- moved R11 0.90 mm to (45.1, 11.4), turned to 90 degrees
Routing:
- net N$43: track 33.7 -> 28.1 mm
- net N$39: track 0.63 -> 2.92 mm
- net N$40: track 18.5 -> 20.1 mm
- net VSUPPLY: track 89.6 -> 88.5 mm
- net N$26: track 3.10 -> 2.08 mm
- net N$37: track 5.87 -> 6.88 mm
Changed lines of the file:
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@@
 <element name="R1" library="rcl" package="0207/7" value="10K" x="16.51" y="50.8"/>
 <element name="R2" library="rcl" package="0207/7" value="7K5" x="12.7" y="47.625" rot="R180"/>
-<element name="C1" library="rcl" package="E3,5-8" value="330uF" x="29.21" y="60.325" rot="R180"/>
+<element name="C1" library="rcl" package="E3,5-8" value="330uF" x="34.29" y="59.69" rot="R45"/>
 <element name="R4" library="rcl" package="0207/7" value="100k" x="31.75" y="30.48" rot="R270"/>
 <element name="T1" library="transistor" package="SOT23" value="" x="5.08" y="14.605" rot="MR180"/>
@@
 <element name="T4" library="transistor" package="SOT23-BEC" value="" x="54.61" y="31.75" rot="MR0"/>
 <element name="D1" library="diode" package="CB417-15" value="P6KEXXC" x="45.72" y="47.625" rot="R90"/>
-<element name="R11" library="rcl" package="R0603" value="15K4" x="45.72" y="10.795" rot="MR180"/>
+<element name="R11" library="rcl" package="R0603" value="15K4" x="45.085" y="11.43" rot="MR90"/>
 <element name="LED2" library="led" package="LED5MM" value="" x="39.37" y="33.02"/>
 <element name="R13" library="rcl" package="0207/7" value="15K4" x="41.275" y="24.765" rot="R90"/>
-<element name="T3" library="transistor" package="SOT23-BEC" value="" x="48.26" y="14.605" rot="MR90"/>
+<element name="T3" library="transistor" package="SOT23-BEC" value="" x="46.355" y="15.24" rot="MR90"/>
 <element name="D2" library="diode" package="CB417-15" value="P6KEXXC" x="45.72" y="27.305" rot="R270"/>
 <element name="R14" library="rcl" package="R0603" value="15K4" x="5.08" y="8.89" rot="MR180"/>
@@
 <attribute name="MPN" value="237-102" x="1529.715" y="7.62" size="1.778" layer="27" rot="R90" display="off"/>
 </element>
-<element name="D11" library="diode" package="CB417-15" value="P6KEXXC" x="58.42" y="11.43" rot="R180"/>
+<element name="D11" library="diode" package="CB417-15" value="P6KEXXC" x="58.42" y="12.7" rot="R180"/>
 <element name="F5" library="fuse" package="TE5" value="" x="63.5" y="5.715">
 <attribute name="OC_FARNELL" value="unknown" x="15.24" y="-1489.075" size="1.778" layer="27" display="off"/>
@@
 <element name="JP7" library="pinhead" package="1X02" value="" x="41.91" y="6.35" rot="R90"/>
 <element name="JP8" library="pinhead" package="1X02" value="" x="41.91" y="16.51" rot="R90"/>
+<element name="H1" library="holes" package="3,0" value="MOUNT-HOLE3.0" x="50.165" y="71.12"/>
+<element name="H2" library="holes" package="3,0" value="MOUNT-HOLE3.0" x="50.165" y="6.35"/>
 </elements>
 <signals>
@@
 <contactref element="LED2" pad="A"/>
 <contactref element="LED1" pad="A"/>
-<wire x1="30.988" y1="60.325" x2="38.1" y2="53.213" width="0.8128" layer="16"/>
-<wire x1="38.1" y1="53.213" x2="38.1" y2="44.45" width="0.8128" layer="16"/>
 <wire x1="38.1" y1="44.45" x2="38.1" y2="38.735" width="0.8128" layer="16"/>
 <wire x1="38.1" y1="38.735" x2="38.1" y2="34.925" width="0.8128" layer="16"/>
@@
 <wire x1="50.8" y1="35.687" x2="50.673" y2="35.56" width="0.8128" layer="16"/>
 <wire x1="50.673" y1="35.56" x2="45.72" y2="35.56" width="0.8128" layer="16"/>
-<wire x1="21.275" y1="64.135" x2="29.21" y2="64.135" width="0.8128" layer="16"/>
-<wire x1="29.21" y1="64.135" x2="30.988" y2="62.357" width="0.8128" layer="16"/>
-<wire x1="30.988" y1="62.357" x2="30.988" y2="60.325" width="0.8128" layer="16"/>
+<wire x1="38.1" y1="44.45" x2="38.1" y2="53.365525" width="0.8128" layer="16"/>
+<wire x1="21.275" y1="64.135" x2="27.305" y2="64.135" width="0.8128" layer="16"/>
+<wire x1="27.305" y1="64.135" x2="33.02" y2="58.42" width="0.8128" layer="16"/>
+<wire x1="38.1" y1="53.365525" x2="33.0327625" y2="58.4327625" width="0.8128" layer="16"/>
 </signal>
 <signal name="N$3">
@@
 <wire x1="41.275" y1="20.955" x2="41.91" y2="20.32" width="0.8128" layer="16"/>
 <wire x1="41.91" y1="20.32" x2="45.72" y2="20.32" width="0.8128" layer="16"/>
-<wire x1="49.36" y1="14.605" x2="50.8" y2="16.045" width="0.8128" layer="16"/>
-<wire x1="50.8" y1="16.045" x2="50.8" y2="19.177" width="0.8128" layer="16"/>
 <wire x1="50.8" y1="19.177" x2="50.292" y2="19.685" width="0.8128" layer="16"/>
 <wire x1="50.292" y1="19.685" x2="45.72" y2="19.685" width="0.8128" layer="16"/>
+<wire x1="47.455" y1="15.24" x2="47.455" y2="17.315" width="0.6096" layer="16"/>
+<wire x1="47.455" y1="17.315" x2="45.72" y2="19.05" width="0.6096" layer="16"/>
+<wire x1="45.72" y1="19.05" x2="45.72" y2="19.685" width="0.6096" layer="16"/>
 </signal>
 <signal name="N$26">
 <contactref element="R11" pad="2"/>
 <contactref element="T3" pad="B"/>
-<wire x1="46.57" y1="10.795" x2="47.16" y2="11.385" width="0.6096" layer="16"/>
-<wire x1="47.16" y1="11.385" x2="47.16" y2="13.655" width="0.6096" layer="16"/>
+<wire x1="45.085" y1="12.28" x2="45.085" y2="14.12" width="0.6096" layer="16"/>
+<wire x1="45.085" y1="14.12" x2="45.255" y2="14.29" width="0.6096" layer="16"/>
 </signal>
 <signal name="LATCH">
@@
 <wire x1="41.91" y1="5.08" x2="41.91" y2="7.62" width="1.4224" layer="16"/>
 <wire x1="41.91" y1="7.62" x2="41.91" y2="10.16" width="1.4224" layer="16"/>
-<wire x1="41.91" y1="10.16" x2="41.91" y2="10.795" width="1.4224" layer="16"/>
-<wire x1="41.91" y1="10.795" x2="41.91" y2="12.7" width="1.4224" layer="16"/>
+<wire x1="41.91" y1="10.16" x2="41.91" y2="12.7" width="1.4224" layer="16"/>
 <wire x1="41.91" y1="12.7" x2="41.91" y2="15.24" width="1.4224" layer="16"/>
 <wire x1="41.91" y1="15.24" x2="41.91" y2="17.78" width="1.4224" layer="16"/>
-<wire x1="44.87" y1="10.795" x2="41.91" y2="10.795" width="0.6096" layer="16"/>
+<wire x1="45.085" y1="10.58" x2="42.33" y2="10.58" width="0.6096" layer="16"/>
+<wire x1="42.33" y1="10.58" x2="41.91" y2="10.16" width="0.6096" layer="16"/>
 </signal>
 <signal name="N$16">
@@
 <wire x1="59.69" y1="72.39" x2="59.69" y2="69.215" width="3.81" layer="16"/>
 <wire x1="59.69" y1="69.215" x2="61.595" y2="67.31" width="3.81" layer="16"/>
-<wire x1="61.595" y1="67.31" x2="62.605" y2="67.31" width="0" layer="19" extent="16-16"/>
+<wire x1="61.595" y1="67.31" x2="62.605" y2="67.31" width="0.6096" layer="16"/>
 </signal>
 <signal name="N$39">
@@
 <contactref element="R19" pad="2"/>
 <wire x1="66.04" y1="73.025" x2="66.675" y2="73.025" width="3.81" layer="16"/>
-<wire x1="66.675" y1="73.025" x2="67.685" y2="73.025" width="0" layer="19" extent="16-16"/>
-<wire x1="65.405" y1="72.39" x2="66.04" y2="73.025" width="0" layer="19" extent="16-16"/>
+<wire x1="66.675" y1="73.025" x2="67.685" y2="73.025" width="0.6096" layer="16"/>
+<wire x1="66.04" y1="73.025" x2="66.04" y2="72.39" width="0.6096" layer="16"/>
+<wire x1="66.04" y1="72.39" x2="65.405" y2="72.39" width="0.6096" layer="16"/>
 </signal>
 <signal name="N$40">
@@
 <wire x1="74.295" y1="68.54" x2="74.295" y2="71.12" width="0.6096" layer="16"/>
 <wire x1="74.295" y1="71.12" x2="74.93" y2="71.12" width="0.6096" layer="16"/>
-<wire x1="68.205" y1="67.31" x2="69.85" y2="67.31" width="0" layer="19" extent="16-16"/>
+<wire x1="68.205" y1="67.31" x2="69.85" y2="67.31" width="0.6096" layer="16"/>
 </signal>
 <signal name="N$43">
@@
 <contactref element="X8" pad="1"/>
 <contactref element="X9" pad="2"/>
-<wire x1="74.295" y1="15.28" x2="69.89" y2="15.28" width="3.81" layer="16"/>
-<wire x1="69.89" y1="15.28" x2="69.85" y2="15.24" width="2.54" layer="16"/>
-<wire x1="66.04" y1="11.43" x2="69.85" y2="11.43" width="3.81" layer="16"/>
-<wire x1="69.85" y1="11.43" x2="69.85" y2="15.24" width="3.81" layer="16"/>
-<wire x1="66.04" y1="19.177" x2="66.04" y2="19.05" width="2.54" layer="16"/>
-<wire x1="66.04" y1="19.05" x2="69.85" y2="15.24" width="3.81" layer="16"/>
-<wire x1="69.85" y1="11.43" x2="73.66" y2="11.43" width="3.81" layer="16"/>
-<wire x1="73.66" y1="11.43" x2="73.66" y2="15.24" width="3.81" layer="16"/>
-<wire x1="73.66" y1="11.43" x2="73.66" y2="10.795" width="3.81" layer="16"/>
-<wire x1="73.66" y1="10.795" x2="66.675" y2="10.795" width="3.81" layer="16"/>
-<wire x1="66.675" y1="10.795" x2="66.04" y2="11.43" width="3.81" layer="16"/>
-<wire x1="73.66" y1="10.795" x2="74.295" y2="10.12" width="0" layer="19" extent="16-16"/>
+<wire x1="66.04" y1="19.177" x2="66.04" y2="15.24" width="3.81" layer="16"/>
+<wire x1="66.04" y1="15.24" x2="66.04" y2="12.7" width="3.81" layer="16"/>
+<wire x1="74.295" y1="10.12" x2="74.295" y2="12.7" width="3.81" layer="16"/>
+<wire x1="74.295" y1="12.7" x2="74.295" y2="15.28" width="3.81" layer="16"/>
+<wire x1="66.04" y1="12.7" x2="74.295" y2="12.7" width="3.81" layer="16"/>
+<wire x1="74.295" y1="15.28" x2="66.04" y2="15.24" width="3.81" layer="16"/>
 </signal>
 <signal name="N$44">

Commit message: Version at first printout
Parts:
- H1, H2: value MOUNT-HOLE3.0 -> MOUNT-HOLE2.8; device holes:3,0 -> holes:2,8
- moved D6 0.64 mm to (59.7, 65.4)
- moved D9 0.64 mm to (65.4, 65.4)
Routing:
- net N$21: track 70.7 -> 54.8 mm
- net N$40: track 20.1 -> 10.7 mm
- net N$39: track 2.92 -> 0.63 mm
- net N$37: track 6.88 -> 7.62 mm
Changed lines of the file:
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@@
 <element name="T1" library="transistor" package="SOT23" value="" x="5.08" y="14.605" rot="MR180"/>
 <element name="K1" library="relay" package="G2RA-SHORTER" value="G2RATE-OJ" x="54.61" y="39.37"/>
-<element name="D6" library="diode" package="CB429-15" value="UF5404" x="59.69" y="64.77" rot="R90"/>
+<element name="D6" library="diode" package="CB429-15" value="UF5404" x="59.69" y="65.405" rot="R90"/>
 <element name="D7" library="diode" package="DO41-7.6" value="1N5819-T" x="13.335" y="60.96" rot="R90"/>
 <element name="C11" library="rcl" package="C050-024X044" value="100n" x="38.1" y="38.735" rot="R180"/>
@@
 <attribute name="MPN" value="" x="73.66" y="32.385" size="1.778" layer="27" display="off"/>
 </element>
-<element name="D9" library="diode" package="CB429-15" value="UF5404" x="65.405" y="64.77" rot="R90"/>
+<element name="D9" library="diode" package="CB429-15" value="UF5404" x="65.405" y="65.405" rot="R90"/>
 <element name="R18" library="rcl" package="R2512" value="0R1" x="65.405" y="67.31" rot="MR0"/>
 <element name="R19" library="rcl" package="R2512" value="0R1" x="70.485" y="73.025" rot="MR0"/>
@@
 <element name="JP7" library="pinhead" package="1X02" value="" x="41.91" y="6.35" rot="R90"/>
 <element name="JP8" library="pinhead" package="1X02" value="" x="41.91" y="16.51" rot="R90"/>
-<element name="H1" library="holes" package="3,0" value="MOUNT-HOLE3.0" x="50.165" y="71.12"/>
-<element name="H2" library="holes" package="3,0" value="MOUNT-HOLE3.0" x="50.165" y="6.35"/>
+<element name="H1" library="holes" package="2,8" value="MOUNT-HOLE2.8" x="50.165" y="71.12"/>
+<element name="H2" library="holes" package="2,8" value="MOUNT-HOLE2.8" x="50.165" y="6.35"/>
 </elements>
 <signals>
@@
 <wire x1="73.7" y1="48.3" x2="71.12" y2="45.72" width="3.81" layer="16"/>
 <wire x1="66.04" y1="51.435" x2="66.04" y2="45.72" width="3.81" layer="16"/>
-<wire x1="66.04" y1="51.435" x2="66.04" y2="52.07" width="3.81" layer="16"/>
-<wire x1="66.04" y1="52.07" x2="66.04" y2="56.515" width="3.81" layer="16"/>
-<wire x1="66.04" y1="56.515" x2="65.405" y2="57.15" width="2.54" layer="16"/>
 <wire x1="74.295" y1="43.14" x2="73.7" y2="43.14" width="3.81" layer="16"/>
 <wire x1="73.7" y1="43.14" x2="71.12" y2="45.72" width="3.81" layer="16"/>
-<wire x1="65.405" y1="57.15" x2="60.96" y2="57.15" width="2.54" layer="16"/>
-<wire x1="59.69" y1="57.15" x2="60.325" y2="57.15" width="2.54" layer="16"/>
-<wire x1="60.325" y1="57.15" x2="60.96" y2="57.15" width="2.54" layer="16"/>
-<wire x1="60.96" y1="57.15" x2="66.04" y2="52.07" width="2.54" layer="16"/>
 <wire x1="63.5" y1="43.18" x2="66.04" y2="45.72" width="2.54" layer="16"/>
 <wire x1="63.5" y1="43.18" x2="64.135" y2="43.815" width="2.54" layer="16"/>
@@
 <wire x1="73.66" y1="43.815" x2="73.025" y2="43.18" width="2.54" layer="16"/>
 <wire x1="73.025" y1="43.18" x2="63.5" y2="43.18" width="2.54" layer="16"/>
-<wire x1="66.04" y1="51.435" x2="60.325" y2="57.15" width="2.54" layer="16"/>
+<wire x1="60.325" y1="57.785" x2="64.77" y2="57.785" width="3.81" layer="16"/>
+<wire x1="66.04" y1="51.435" x2="66.04" y2="57.15" width="3.81" layer="16"/>
+<wire x1="66.04" y1="57.15" x2="65.405" y2="57.785" width="3.81" layer="16"/>
+<wire x1="60.325" y1="57.785" x2="59.69" y2="57.785" width="0" layer="19" extent="16-16"/>
+<wire x1="65.405" y1="57.785" x2="64.77" y2="57.785" width="0" layer="19" extent="16-16"/>
 </signal>
 <signal name="N$30">
@@
 <contactref element="D6" pad="A"/>
 <contactref element="R18" pad="2"/>
-<wire x1="59.69" y1="72.39" x2="59.69" y2="69.215" width="3.81" layer="16"/>
-<wire x1="59.69" y1="69.215" x2="61.595" y2="67.31" width="3.81" layer="16"/>
-<wire x1="61.595" y1="67.31" x2="62.605" y2="67.31" width="0.6096" layer="16"/>
+<wire x1="59.69" y1="73.025" x2="59.69" y2="67.31" width="3.81" layer="16"/>
+<wire x1="59.69" y1="67.31" x2="61.595" y2="67.31" width="3.81" layer="16"/>
+<wire x1="61.595" y1="67.31" x2="62.605" y2="67.31" width="0" layer="19" extent="16-16"/>
 </signal>
 <signal name="N$39">
@@
 <contactref element="R19" pad="2"/>
 <wire x1="66.04" y1="73.025" x2="66.675" y2="73.025" width="3.81" layer="16"/>
-<wire x1="66.675" y1="73.025" x2="67.685" y2="73.025" width="0.6096" layer="16"/>
-<wire x1="66.04" y1="73.025" x2="66.04" y2="72.39" width="0.6096" layer="16"/>
-<wire x1="66.04" y1="72.39" x2="65.405" y2="72.39" width="0.6096" layer="16"/>
+<wire x1="66.675" y1="73.025" x2="67.685" y2="73.025" width="0" layer="19" extent="16-16"/>
+<wire x1="65.405" y1="73.025" x2="66.04" y2="73.025" width="0" layer="19" extent="16-16"/>
 </signal>
 <signal name="N$40">
@@
 <contactref element="R19" pad="1"/>
 <contactref element="X7" pad="2"/>
-<wire x1="71.755" y1="67.31" x2="69.85" y2="67.31" width="3.81" layer="16"/>
-<wire x1="71.755" y1="67.31" x2="75.565" y2="71.12" width="3.81" layer="16"/>
-<wire x1="75.565" y1="71.12" x2="75.565" y2="73.66" width="3.81" layer="16"/>
-<wire x1="75.565" y1="73.66" x2="74.93" y2="73.66" width="3.81" layer="16"/>
-<wire x1="74.93" y1="73.66" x2="74.93" y2="72.39" width="3.81" layer="16"/>
-<wire x1="74.93" y1="72.39" x2="74.93" y2="71.12" width="3.81" layer="16"/>
-<wire x1="73.285" y1="73.025" x2="73.285" y2="72.39" width="0.6096" layer="16"/>
-<wire x1="73.285" y1="72.39" x2="74.93" y2="72.39" width="0.6096" layer="16"/>
-<wire x1="74.295" y1="68.54" x2="74.295" y2="71.12" width="0.6096" layer="16"/>
-<wire x1="74.295" y1="71.12" x2="74.93" y2="71.12" width="0.6096" layer="16"/>
-<wire x1="68.205" y1="67.31" x2="69.85" y2="67.31" width="0.6096" layer="16"/>
+<wire x1="74.93" y1="73.025" x2="74.295" y2="73.025" width="3.81" layer="16"/>
+<wire x1="74.93" y1="73.025" x2="74.93" y2="68.58" width="3.81" layer="16"/>
+<wire x1="74.295" y1="68.54" x2="71.715" y2="68.54" width="3.81" layer="16"/>
+<wire x1="71.715" y1="68.54" x2="70.485" y2="67.31" width="3.81" layer="16"/>
+<wire x1="70.485" y1="67.31" x2="69.215" y2="67.31" width="3.81" layer="16"/>
+<wire x1="74.295" y1="73.025" x2="73.285" y2="73.025" width="0" layer="19" extent="16-16"/>
+<wire x1="74.295" y1="68.54" x2="74.93" y2="68.58" width="0" layer="19" extent="16-16"/>
+<wire x1="68.205" y1="67.31" x2="69.215" y2="67.31" width="0" layer="19" extent="16-16"/>
 </signal>
 <signal name="N$43">
