File: LockSequencer.sch (EAGLE design)
At the start: 37 parts, among them IC1 4017D, IC2 NE555, K1 G2RA, K2 G2RA

Commit message: Complete versions of the SPICE and Eagle schmatic
Parts:
- removed C10: 100n, rcl:C-EU025-024X044
- removed C8: 10n, rcl:C-EU025-024X044
- removed D5: 1N4004, diode:1N4004
- removed F1, F2: FUSEKS9V, fuse:FUSEKS9V
- removed JP2, JP3, JP4: (no value), pinhead:PINHD-2X2
- removed X2, X3: (no value), con-wago-500:W237-102
- added C11, C14: 100n, rcl:C-EU050-024X044
- added C12: 10n, rcl:C-EUC1206K
- added C13: 10uF, rcl:CPOL-EUE2-5
- added D11, D8: P6KEXXC, diode:P6KEXXC
- added D6, D9: UF5404, diode:SCHOTTKY-DIODECB429-15
- added D7: 1N5819-T, diode:1N5819-T
- added F3, F4, F5, F6: (no value), fuse:TE5
- added JP5, JP6, JP7: (no value), pinhead:PINHD-2X2
- added LED1, LED2, LED3, LED4: (no value), led:LED5MM
- added R10, R11, R14, R16: 15K4, rcl:R-EU_R0603
- added R12, R15, R17: 2K2, rcl:R-EU_0207/7
- added R13: 15K4, rcl:R-EU_0207/7
- added R18, R19: 0R1, rcl:R-EU_R2512
- added R20: 7K5, rcl:R-EU_0207/7
- added R6, R7: 10K, rcl:R-EU_R0805
- added R8: 2K2, rcl:R-EU_R0402
- added R9: 196R, rcl:R-EU_R0805
- added T4: (no value), transistor:MMBTA42LT1-NPN-SOT23-BEC
- added T5: (no value), transistor:-NPN_DRIVER-
- added U$1, U$13: 2N7002, transistor-fet:2N7002
- added X4, X5, X6, X7, X8, X9: (no value), con-wago-500:W237-102
- C1: value 100uF -> 330uF; device rcl:CPOL-EU085CS-1AR -> rcl:CPOL-EUE3.5-8
- C2: value 100n -> 100uF; device rcl:C-EU025-024X044 -> rcl:CPOL-EUE2-5
- C3, C5: device rcl:C-EU025-024X044 -> rcl:C-EUC1206K
- C4: device rcl:C-EU025-024X044 -> rcl:C-EU050-024X044
- C6: value 1u -> 1uF; device rcl:CPOL-EU085CS-1AR -> rcl:C-EUC1206K
- C7: value 10n -> 100n; device rcl:C-EU025-024X044 -> rcl:C-EUC1206K
- C9: value 100uF -> 100n; device rcl:CPOL-EU085CS-1AR -> rcl:C-EUC1206K
- D1, D2: value 1N4004 -> P6KEXXC; device diode:1N4004 -> diode:P6KEXXC
- D3: value Z3.6V -> Z12V; device diode:DIODE-SOD323-R -> diode:DIODE-SOD323-W
- K1, K2: value G2RA -> G2RATE-OJ; device relay:G2RA -> relay:G2RATE-OJ
- R1: value 10k -> 10K; device rcl:R-EU_0204/2V -> rcl:R-EU_0207/7
- R2: value 10k -> 7K5; device rcl:R-EU_0204/2V -> rcl:R-EU_0207/7
- R3: value 100k -> (none); device rcl:R-EU_0204/2V -> pot:TRIM_EU-CA9V
- R4: device rcl:R-EU_0204/2V -> rcl:R-EU_0207/7
- R5: value 1k -> 2K2; device rcl:R-EU_0204/2V -> rcl:R-EU_R0402
- T2, T3: device transistor:-NPN_DRIVER- -> transistor:MMBTA42LT1-NPN-SOT23-BEC
Connections:
- removed net +12V: C10.1, C4.1, C7.1, C8.1, C9.+, D1.A, D1.C, D2.C, D4.C, D5.C, IC2./RES, IC2.VCC+, K11.1, K11.2, K21.1, R1.2, R4.2, R5.2, T1.C, X1-1.KL, X2-2.KL, X3-2.KL
- removed net N$19: C8.2, D5.A, F1.1, X3-1.KL
- new net N$23: R5.1, U$13.G
- new net N$24: IC2.DIS, R3.A, R3.S, R4.1
- new net N$25: C7.1, D3.C, R9.1, T2.B
- new net N$26: R11.2, T3.B
- new net N$27: D1.1, K11.2, LED1.C, T4.C
- new net N$28: R8.2, U$1.G
- new net N$29: LED1.A, R12.1
- new net N$30: F4.2, X5-1.KL
- new net N$31: F3.2, X6-1.KL
- new net N$32: JP5.1, JP5.2, JP6.1, JP6.2, JP7.1, JP7.2, R10.1
- new net N$33: JP5.3, JP5.4, JP6.3, JP6.4, JP7.3, JP7.4, R11.1
- new net N$34: LED3.A, R15.1
- new net N$35: LED3.C, T1.C
- new net N$36: R16.1, T5.B
- new net N$37: D6.A, R18.2
- new net N$38: LED4.C, T5.C
- new net N$39: D9.A, R19.2
- new net N$40: R18.1, R19.1, X7-2.KL
- new net N$43: D11.2, K22.P, X8-2.KL, X9-2.KL
- new net N$44: F6.2, X8-1.KL
- new net N$45: F5.2, X9-1.KL
- new net RESET_N: IC2./RES, R7.1, U$1.D
- new net VDD: C13.+, C14.1, C3.1, C4.1, IC2.VCC+, R1.2, R15.2, R17.2, R4.2, R6.2, R7.2, T2.E
- new net VEXTERNAL: D4.A, D7.A, K12.S, K22.S, X1-1.KL, X4-1.KL, X4-2.KL
- new net VSS: C3.2
- new net VSUPPLY: C1.+, C11.1, D1.2, D2.2, D7.C, K11.1, K21.1, R12.2, R13.2, R9.2, T2.C
- net GND: now also C11.2, C12.2, C13.-, C14.2, C2.-, C6.2, C7.2, C9.2, D11.1, D8.1, F3.1, F4.1, F5.1, F6.1, R20.1, T4.E, T5.E, U$1.S, U$13.S, X7-1.KL; no longer C10.2, C2.2, C3.2, C6.-, C9.-, K12.P, K22.P, T2.E
- net N$14: now also C6.1, IC2.TRE, IC2.TRI, R3.E; no longer C6.+, IC2.DIS, R3.1, R4.1
- net N$15: now also R10.2, T4.B; no longer IC2.TRE, IC2.TRI, R3.2
- net N$16: now also R14.1; no longer JP2.1, JP2.2, JP3.1, JP3.2, JP4.1, JP4.2
- net N$17: now also LED4.A, R17.1; no longer JP2.3, JP2.4, JP3.3, JP3.4, JP4.3, JP4.4, T3.B
- net N$18: now also D2.1, LED2.C; no longer D2.A
- net N$2: now also C2.+, C9.1; no longer C1.+, C2.1, D3.C
- net N$20: now also D4.C, R20.2; no longer C7.2, D4.A, F2.1, X2-1.KL
- net N$21: now also D6.C, D8.2, D9.C, K12.P, X5-2.KL, X6-2.KL; no longer F2.2, K12.S
- net N$22: now also LED2.A, R13.1; no longer F1.2, K22.S
- net N$3: now also C12.1, R5.2; no longer T2.B
- net N$4: now also R14.2
- net N$5: now also R16.2
- net RESET: now also R6.1, R8.1, U$13.D; no longer C3.1, R5.1, T2.C
Other:
- moved on the sheet: C1, C3, C4, C5, C7, D3, D4, IC1, IC2, JP1, K1, K2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

Commit message: Initial Component placement, removed current sinking to detect polarity
Parts:
- removed D4: 1N4004, diode:1N4004
- removed R20: 7K5, rcl:R-EU_0207/7
- removed X4: (no value), con-wago-500:W237-102
- added F1: (no value), fuse:TE5
- added X2, X3: (no value), con-wago-500:W237-102
- R12, R13, R15, R17: device rcl:R-EU_0207/7 -> rcl:R-EU_0207/2V
- R3: value (none) -> 220K
Connections:
- removed net GND: C1.-, C11.2, C12.2, C13.-, C14.2, C2.-, C4.2, C5.2, C6.2, C7.2, C9.2, D11.1, D3.A, D8.1, F3.1, F4.1, F5.1, F6.1, IC2.GND, R2.1, R20.1, T1.E, T3.E, T4.E, T5.E, U$1.S, U$13.S, U$4.GND, X1-2.KL, X7-1.KL
- removed net N$20: D4.C, R20.2
- new net N$19: D7.A, F1.1
- net N$43: now also X8-1.KL; no longer X8-2.KL
- net N$44: now also X8-2.KL; no longer X8-1.KL
- net VDD: now also IC1P.VDD
- net VEXTERNAL: now also F1.2, X2-1.KL, X2-2.KL, X3-1.KL; no longer D4.A, D7.A, X1-1.KL, X4-1.KL, X4-2.KL
- net VSS: now also C1.-, C11.2, C12.2, C13.-, C14.2, C2.-, C4.2, C5.2, C6.2, C7.2, C9.2, D11.1, D3.A, D8.1, F3.1, F4.1, F5.1, F6.1, IC1P.VSS, IC2.GND, R2.1, T1.E, T3.E, T4.E, T5.E, U$1.S, U$13.S, U$4.GND, X1-1.KL, X1-2.KL, X3-2.KL, X7-1.KL
Other:
- moved on the sheet: C3, X1-1, X1-2, X8-1, X8-2

Commit message: Initial component placement prior to first auto routing attempt
Parts:
- removed X1, X3: (no value), con-wago-500:W237-102
- added JP2, JP3: (no value), pinhead:PINHD-1X8
- added JP4, JP8: (no value), pinhead:PINHD-1X2
- added R20: 100k, rcl:R-EU_0207/7
- added X10: (no value), con-wago-500:W237-103
- JP1: device pinhead:PINHD-2X9 -> pinhead:PINHD-1X2
- JP5, JP6, JP7: device pinhead:PINHD-2X2 -> pinhead:PINHD-1X2
- R15: device rcl:R-EU_0207/2V -> rcl:R-EU_0207/7
- X2: device con-wago-500:W237-102 -> con-wago-500:W237-103
Connections:
- removed net N$34: LED3.A, R15.1
- removed net N$35: LED3.C, T1.C
- removed net N$38: LED4.C, T5.C
- new net LATCH: JP1.1, JP1.2, JP4.1, JP4.2, JP6.1, JP6.2, R10.1
- new net N$20: IC1A.Q0, R16.2
- new net OPEN: JP5.1, JP5.2, JP7.1, JP7.2, JP8.1, JP8.2, R11.1
- net N$10: now also IC1A.Q6, JP2.6, JP3.6; no longer IC1A.Q5, JP1.11, JP1.12
- net N$11: now also IC1A.Q7, JP2.7, JP3.7; no longer IC1A.Q6, JP1.13, JP1.14
- net N$12: now also IC1A.Q8, JP2.8, JP3.8; no longer IC1A.Q7, JP1.15, JP1.16
- net N$13: now also LED4.C, R17.1; no longer IC1A.Q8, JP1.17, JP1.18
- net N$14: now also R20.1, R3.A; no longer R3.E
- net N$17: now also R17.2, T5.C; no longer LED4.A, R17.1
- net N$24: now also R20.2, R3.E; no longer R3.A
- net N$32: now also LED3.C, R15.2; no longer JP5.1, JP5.2, JP6.1, JP6.2, JP7.1, JP7.2, R10.1
- net N$33: now also R15.1, T1.C; no longer JP5.3, JP5.4, JP6.3, JP6.4, JP7.3, JP7.4, R11.1
- net N$5: now also IC1A.Q1, JP2.1, JP3.1; no longer IC1A.Q0, JP1.1, JP1.2, R16.2
- net N$6: now also IC1A.Q2, JP2.2, JP3.2; no longer IC1A.Q1, JP1.3, JP1.4
- net N$7: now also IC1A.Q3, JP2.3, JP3.3; no longer IC1A.Q2, JP1.5, JP1.6
- net N$8: now also IC1A.Q4, JP2.4, JP3.4; no longer IC1A.Q3, JP1.7, JP1.8
- net N$9: now also IC1A.Q5, JP2.5, JP3.5; no longer IC1A.Q4, JP1.10, JP1.9
- net VDD: now also LED3.A, LED4.A; no longer R15.2, R17.2
- net VEXTERNAL: now also X10-1.KL, X10-2.KL, X10-3.KL; no longer X2-1.KL, X2-2.KL, X3-1.KL
- net VSS: now also X2-1.KL, X2-2.KL, X2-3.KL; no longer X1-1.KL, X1-2.KL, X3-2.KL
Other:
- moved on the sheet: C6, LED3, LED4, R11, R15, R17, R3, R4, T3, X2-1, X2-2

Commit message: Tweaked positions
Parts:
- R17: device rcl:R-EU_0207/2V -> rcl:R-EU_0207/7
Connections:
- net N$21: now also X5-1.KL; no longer X5-2.KL
- net N$30: now also X5-2.KL; no longer X5-1.KL
- net N$43: now also X8-2.KL; no longer X8-1.KL
- net N$44: now also X8-1.KL; no longer X8-2.KL
Other:
- moved on the sheet: X5-1, X5-2, X8-1, X8-2
Changed lines of the file:
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@@
 <part name="R16" library="rcl" deviceset="R-EU_" device="R0603" value="15K4"/>
 <part name="LED4" library="led" deviceset="LED" device="5MM"/>
-<part name="R17" library="rcl" deviceset="R-EU_" device="0207/2V" value="2K2"/>
+<part name="R17" library="rcl" deviceset="R-EU_" device="0207/7" value="2K2"/>
 <part name="K2" library="relay" deviceset="G2RA" device="TE-OJ" value="G2RATE-OJ"/>
 <part name="X5" library="con-wago-500" deviceset="W237-102" device=""/>
@@
 <instance part="K2" gate="1" x="330.2" y="66.04"/>
 <instance part="K2" gate="2" x="347.98" y="71.12"/>
-<instance part="X5" gate="-1" x="350.52" y="109.22" rot="R180"/>
-<instance part="X5" gate="-2" x="350.52" y="111.76" rot="R180"/>
+<instance part="X5" gate="-1" x="350.52" y="111.76" rot="R180"/>
+<instance part="X5" gate="-2" x="350.52" y="109.22" rot="R180"/>
 <instance part="X6" gate="-1" x="360.68" y="109.22" rot="R180"/>
 <instance part="X6" gate="-2" x="360.68" y="111.76" rot="R180"/>
@@
 <instance part="X7" gate="-1" x="403.86" y="104.14" rot="R180"/>
 <instance part="X7" gate="-2" x="403.86" y="109.22" rot="R180"/>
-<instance part="X8" gate="-1" x="355.6" y="55.88" rot="R180"/>
-<instance part="X8" gate="-2" x="355.6" y="53.34" rot="R180"/>
+<instance part="X8" gate="-1" x="355.6" y="53.34" rot="R180"/>
+<instance part="X8" gate="-2" x="355.6" y="55.88" rot="R180"/>
 <instance part="X9" gate="-1" x="365.76" y="53.34" rot="R180"/>
 <instance part="X9" gate="-2" x="365.76" y="55.88" rot="R180"/>
@@
 <segment>
 <pinref part="K1" gate="2" pin="P"/>
-<pinref part="X5" gate="-2" pin="KL"/>
 <wire x1="342.9" y1="121.92" x2="342.9" y2="119.38" width="0.1524" layer="91"/>
 <wire x1="342.9" y1="119.38" x2="342.9" y2="111.76" width="0.1524" layer="91"/>
-<wire x1="342.9" y1="111.76" x2="345.44" y2="111.76" width="0.1524" layer="91"/>
 <pinref part="X6" gate="-2" pin="KL"/>
 <wire x1="342.9" y1="119.38" x2="355.6" y2="119.38" width="0.1524" layer="91"/>
@@
 <wire x1="375.92" y1="127" x2="370.84" y2="127" width="0.1524" layer="91"/>
 <wire x1="370.84" y1="127" x2="370.84" y2="119.38" width="0.1524" layer="91"/>
+<pinref part="X5" gate="-1" pin="KL"/>
+<wire x1="342.9" y1="111.76" x2="345.44" y2="111.76" width="0.1524" layer="91"/>
 </segment>
 </net>
 <net name="N$30" class="0">
 <segment>
-<pinref part="X5" gate="-1" pin="KL"/>
-<wire x1="345.44" y1="109.22" x2="342.9" y2="109.22" width="0.1524" layer="91"/>
 <pinref part="F4" gate="1" pin="2"/>
 <wire x1="342.9" y1="106.68" x2="342.9" y2="109.22" width="0.1524" layer="91"/>
+<pinref part="X5" gate="-2" pin="KL"/>
+<wire x1="345.44" y1="109.22" x2="342.9" y2="109.22" width="0.1524" layer="91"/>
 </segment>
 </net>
@@
 <wire x1="375.92" y1="53.34" x2="375.92" y2="63.5" width="0.1524" layer="91"/>
 <pinref part="K2" gate="2" pin="P"/>
-<pinref part="X8" gate="-1" pin="KL"/>
+<pinref part="X8" gate="-2" pin="KL"/>
 <wire x1="350.52" y1="55.88" x2="347.98" y2="55.88" width="0.1524" layer="91"/>
 </segment>
@@
 <pinref part="F6" gate="1" pin="2"/>
 <wire x1="347.98" y1="50.8" x2="347.98" y2="53.34" width="0.1524" layer="91"/>
-<pinref part="X8" gate="-2" pin="KL"/>
+<pinref part="X8" gate="-1" pin="KL"/>
 <wire x1="350.52" y1="53.34" x2="347.98" y2="53.34" width="0.1524" layer="91"/>
 </segment>

Commit message: 555 and 4017 nearly sorted out
Parts:
- R12: device rcl:R-EU_0207/2V -> rcl:R-EU_0207/7
- R17: device rcl:R-EU_0207/7 -> rcl:R-EU_0309/12
- R6: device rcl:R-EU_R0805 -> rcl:R-EU_0207/7
Changed lines of the file:
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@@
 <part name="R5" library="rcl" deviceset="R-EU_" device="R0402" value="2K2"/>
 <part name="U$13" library="transistor-fet" deviceset="2N7002" device=""/>
-<part name="R6" library="rcl" deviceset="R-EU_" device="R0805" value="10K"/>
+<part name="R6" library="rcl" deviceset="R-EU_" device="0207/7" value="10K"/>
 <part name="U$1" library="transistor-fet" deviceset="2N7002" device=""/>
 <part name="R7" library="rcl" deviceset="R-EU_" device="R0805" value="10K"/>
@@
 <part name="R10" library="rcl" deviceset="R-EU_" device="R0603" value="15K4"/>
 <part name="LED1" library="led" deviceset="LED" device="5MM"/>
-<part name="R12" library="rcl" deviceset="R-EU_" device="0207/2V" value="2K2"/>
+<part name="R12" library="rcl" deviceset="R-EU_" device="0207/7" value="2K2"/>
 <part name="T4" library="transistor" deviceset="*-NPN-" device="SOT23-BEC" technology="MMBTA42LT1"/>
 <part name="D1" library="diode" deviceset="P6KEXXC" device=""/>
@@
 <part name="R16" library="rcl" deviceset="R-EU_" device="R0603" value="15K4"/>
 <part name="LED4" library="led" deviceset="LED" device="5MM"/>
-<part name="R17" library="rcl" deviceset="R-EU_" device="0207/7" value="2K2"/>
+<part name="R17" library="rcl" deviceset="R-EU_" device="0309/12" value="2K2"/>
 <part name="K2" library="relay" deviceset="G2RA" device="TE-OJ" value="G2RATE-OJ"/>
 <part name="X5" library="con-wago-500" deviceset="W237-102" device=""/>
@@
 </segment>
 </net>
-<net name="N$5" class="0">
-<segment>
-<wire x1="236.22" y1="76.2" x2="228.6" y2="76.2" width="0.1524" layer="91"/>
-<pinref part="JP2" gate="A" pin="1"/>
-<pinref part="JP3" gate="A" pin="1"/>
-<pinref part="IC1" gate="A" pin="Q1"/>
-<wire x1="228.6" y1="76.2" x2="210.82" y2="76.2" width="0.1524" layer="91"/>
-<junction x="228.6" y="76.2"/>
-</segment>
-</net>
-<net name="N$6" class="0">
-<segment>
-<wire x1="236.22" y1="73.66" x2="228.6" y2="73.66" width="0.1524" layer="91"/>
-<pinref part="JP2" gate="A" pin="2"/>
-<pinref part="JP3" gate="A" pin="2"/>
-<pinref part="IC1" gate="A" pin="Q2"/>
-<wire x1="210.82" y1="73.66" x2="228.6" y2="73.66" width="0.1524" layer="91"/>
-<junction x="228.6" y="73.66"/>
-</segment>
-</net>
 <net name="N$7" class="0">
 <segment>
@@
 <pinref part="JP3" gate="A" pin="3"/>
 <pinref part="IC1" gate="A" pin="Q3"/>
-<wire x1="228.6" y1="71.12" x2="210.82" y2="71.12" width="0.1524" layer="91"/>
+<wire x1="210.82" y1="71.12" x2="228.6" y2="71.12" width="0.1524" layer="91"/>
 <junction x="228.6" y="71.12"/>
-</segment>
-</net>
-<net name="N$8" class="0">
-<segment>
-<wire x1="236.22" y1="68.58" x2="228.6" y2="68.58" width="0.1524" layer="91"/>
-<pinref part="JP2" gate="A" pin="4"/>
-<pinref part="JP3" gate="A" pin="4"/>
-<pinref part="IC1" gate="A" pin="Q4"/>
-<wire x1="210.82" y1="68.58" x2="228.6" y2="68.58" width="0.1524" layer="91"/>
-<junction x="228.6" y="68.58"/>
 </segment>
 </net>
@@
 <wire x1="210.82" y1="66.04" x2="228.6" y2="66.04" width="0.1524" layer="91"/>
 <junction x="228.6" y="66.04"/>
-</segment>
-</net>
-<net name="N$10" class="0">
-<segment>
-<wire x1="236.22" y1="63.5" x2="228.6" y2="63.5" width="0.1524" layer="91"/>
-<pinref part="JP2" gate="A" pin="6"/>
-<pinref part="JP3" gate="A" pin="6"/>
-<pinref part="IC1" gate="A" pin="Q6"/>
-<wire x1="210.82" y1="63.5" x2="228.6" y2="63.5" width="0.1524" layer="91"/>
-<junction x="228.6" y="63.5"/>
-</segment>
-</net>
-<net name="N$11" class="0">
-<segment>
-<wire x1="236.22" y1="60.96" x2="228.6" y2="60.96" width="0.1524" layer="91"/>
-<pinref part="JP2" gate="A" pin="7"/>
-<pinref part="JP3" gate="A" pin="7"/>
-<pinref part="IC1" gate="A" pin="Q7"/>
-<wire x1="210.82" y1="60.96" x2="228.6" y2="60.96" width="0.1524" layer="91"/>
-<junction x="228.6" y="60.96"/>
 </segment>
 </net>
@@
 </segment>
 </net>
-<net name="VSUPPLY" class="0">
+<net name="VSUPPLY" class="1">
 <segment>
 <pinref part="C1" gate="G$1" pin="+"/>
@@
 </segment>
 </net>
-<net name="VDD" class="0">
+<net name="VDD" class="1">
 <segment>
 <pinref part="R6" gate="G$1" pin="2"/>
@@
 </segment>
 </net>
-<net name="VSS" class="0">
+<net name="VSS" class="3">
 <segment>
 <pinref part="C1" gate="G$1" pin="-"/>
@@
 </segment>
 </net>
+<net name="N$34" class="0">
+<segment>
+<pinref part="IC1" gate="A" pin="Q1"/>
+<wire x1="236.22" y1="76.2" x2="228.6" y2="76.2" width="0.1524" layer="91"/>
+<pinref part="JP2" gate="A" pin="1"/>
+<pinref part="JP3" gate="A" pin="1"/>
+<wire x1="210.82" y1="76.2" x2="228.6" y2="76.2" width="0.1524" layer="91"/>
+<junction x="228.6" y="76.2"/>
+</segment>
+</net>
+<net name="N$35" class="0">
+<segment>
+<pinref part="IC1" gate="A" pin="Q2"/>
+<wire x1="236.22" y1="73.66" x2="228.6" y2="73.66" width="0.1524" layer="91"/>
+<pinref part="JP2" gate="A" pin="2"/>
+<pinref part="JP3" gate="A" pin="2"/>
+<wire x1="210.82" y1="73.66" x2="228.6" y2="73.66" width="0.1524" layer="91"/>
+<junction x="228.6" y="73.66"/>
+</segment>
+</net>
+<net name="N$5" class="0">
+<segment>
+<pinref part="IC1" gate="A" pin="Q6"/>
+<wire x1="236.22" y1="63.5" x2="228.6" y2="63.5" width="0.1524" layer="91"/>
+<pinref part="JP2" gate="A" pin="6"/>
+<pinref part="JP3" gate="A" pin="6"/>
+<wire x1="210.82" y1="63.5" x2="228.6" y2="63.5" width="0.1524" layer="91"/>
+<junction x="228.6" y="63.5"/>
+</segment>
+</net>
+<net name="N$6" class="0">
+<segment>
+<pinref part="IC1" gate="A" pin="Q7"/>
+<wire x1="236.22" y1="60.96" x2="228.6" y2="60.96" width="0.1524" layer="91"/>
+<pinref part="JP2" gate="A" pin="7"/>
+<pinref part="JP3" gate="A" pin="7"/>
+<wire x1="210.82" y1="60.96" x2="228.6" y2="60.96" width="0.1524" layer="91"/>
+<junction x="228.6" y="60.96"/>
+</segment>
+</net>
+<net name="N$38" class="0">
+<segment>
+<pinref part="IC1" gate="A" pin="Q4"/>
+<wire x1="236.22" y1="68.58" x2="228.6" y2="68.58" width="0.1524" layer="91"/>
+<pinref part="JP2" gate="A" pin="4"/>
+<pinref part="JP3" gate="A" pin="4"/>
+<wire x1="210.82" y1="68.58" x2="228.6" y2="68.58" width="0.1524" layer="91"/>
+<junction x="228.6" y="68.58"/>
+</segment>
+</net>

Commit message: Routing completed
Parts:
- R13: device rcl:R-EU_0207/2V -> rcl:R-EU_0207/7
Connections:
- removed net N$22 (its old number): LED2.A, R13.1
- removed net N$29: LED1.A, R12.1
- removed net N$31: F3.2, X6-1.KL
- new net N$10: LED1.C, R12.2
- new net N$11: F3.2, X6-2.KL
- new net N$8: LED2.C, R13.2
- net N$18: now also K21.1, R13.1; no longer K21.2, LED2.C
- net N$21: now also X5-2.KL, X6-1.KL; no longer X5-1.KL, X6-2.KL
- net N$27: now also R12.1; no longer LED1.C
- net N$30: now also X5-1.KL; no longer X5-2.KL
- net N$43: now also K22.S, X8-1.KL; no longer K22.P, X8-2.KL
- net N$44: now also X8-2.KL; no longer X8-1.KL
- net VEXTERNAL: now also K22.P; no longer K22.S
- net VSUPPLY: now also K21.2, LED1.A, LED2.A; no longer K21.1, R12.2, R13.2
Other:
- moved on the sheet: K1, K2, LED1, LED2, R12, R13, X5-1, X5-2, X6-1, X6-2, X8-1, X8-2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

Commit message: Final tweaks to layout
Parts:
- added H1, H2: MOUNT-HOLE3.0, holes:MOUNT-HOLE3.0
Changed lines of the file:
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@@
 <part name="JP7" library="pinhead" deviceset="PINHD-1X2" device=""/>
 <part name="JP8" library="pinhead" deviceset="PINHD-1X2" device=""/>
+<part name="H1" library="holes" deviceset="MOUNT-HOLE" device="3.0"/>
+<part name="H2" library="holes" deviceset="MOUNT-HOLE" device="3.0"/>
 </parts>
 <sheets>
@@
 <instance part="JP7" gate="G$1" x="251.46" y="53.34" rot="R180"/>
 <instance part="JP8" gate="G$1" x="251.46" y="45.72" rot="R180"/>
+<instance part="H1" gate="G$1" x="302.26" y="165.1"/>
+<instance part="H2" gate="G$1" x="330.2" y="165.1"/>
 </instances>
 <busses>

Commit message: Version at first printout
Parts:
- H1, H2: value MOUNT-HOLE3.0 -> MOUNT-HOLE2.8; device holes:MOUNT-HOLE3.0 -> holes:MOUNT-HOLE2.8
Changed lines of the file:
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@@
 <part name="JP7" library="pinhead" deviceset="PINHD-1X2" device=""/>
 <part name="JP8" library="pinhead" deviceset="PINHD-1X2" device=""/>
-<part name="H1" library="holes" deviceset="MOUNT-HOLE" device="3.0"/>
-<part name="H2" library="holes" deviceset="MOUNT-HOLE" device="3.0"/>
+<part name="H1" library="holes" deviceset="MOUNT-HOLE" device="2.8" value="MOUNT-HOLE2.8"/>
+<part name="H2" library="holes" deviceset="MOUNT-HOLE" device="2.8" value="MOUNT-HOLE2.8"/>
 </parts>
 <sheets>
